Commit message: added lidar test

File: simple_driving/resources/simplecar.urdf (robot description, URDF)
Before this commit: robot simplecar, 7 links, 6 joints
Links:
- added link lidar_link, mass 0.1; collision box size=0.1 0.1 0.1; visual box size=0.1 0.1 0.1
Joints:
- added joint base_to_lidar: type fixed, parent base_link, child lidar_link, origin xyz=0 0 0.1 rpy=0 0 0
